File: AdapterPCB/adapter/proj/adapter.kicad_pcb (KiCad board)
At the start: 2 copper layers, 66 x 67 mm, 37 parts, among them J2 VGA, U1 SN74LVC245APW, U2 SN74LVC245APW

Commit message: ye
Parts:
- moved G*** 2.88 mm to (118.6, 103.6)
Other:
- board text added: "By swr06"
- board text added: "VGA PMOD Adapter"
Changed lines of the file:
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@@
 	(footprint "LOGO:LOGOSS"
 		(layer "F.Cu")
-		(at 117.856 106.426)
+		(at 118.5672 103.632)
 		(property "Reference" "G***"
 			(at 0 0 0)
@@
 	)
 	(gr_rect
+		(start 112.8268 46.5836)
+		(end 117.9576 67.31)
+		(stroke
+			(width 0.1)
+			(type default)
+		)
+		(fill no)
+		(layer "F.SilkS")
+	)
+	(gr_rect
 		(start 111.76 45.512)
 		(end 177.8 112.522)
@@
 		)
 	)
+	(gr_text "330"
+		(at 119.6848 96.266 0)
+		(layer "F.SilkS")
+		(effects
+			(font
+				(size 0.5 0.5)
+				(thickness 0.1)
+			)
+			(justify left bottom)
+		)
+	)
 	(gr_text "x"
 		(at 146.685 105.791 0)
@@
 		)
 	)
+	(gr_text "330"
+		(at 155.2956 96.1644 0)
+		(layer "F.SilkS")
+		(effects
+			(font
+				(size 0.5 0.5)
+				(thickness 0.1)
+			)
+			(justify left bottom)
+		)
+	)
 	(gr_text "gnd"
 		(at 156.972 57.404 0)
@@
 	)
 	(gr_text "Peak"
-		(at 170.942 99.314 270)
+		(at 171.704 99.7712 270)
 		(layer "F.SilkS")
 		(effects
@@
 	)
 	(gr_text "< p1"
-		(at 166.935 59.182 0)
+		(at 167.405 59.268 0)
 		(layer "F.SilkS")
 		(effects
@@
 		)
 	)
+	(gr_text "By swr06"
+		(at 117.1448 56.5912 90)
+		(layer "F.SilkS")
+		(effects
+			(font
+				(size 1.4 1.4)
+				(thickness 0.175)
+			)
+			(justify left bottom)
+		)
+	)
 	(gr_text "gnd"
 		(at 152.146 52.451 90)
@@
 		)
 	)
+	(gr_text "330"
+		(at 136.4488 96.2152 0)
+		(layer "F.SilkS")
+		(effects
+			(font
+				(size 0.5 0.5)
+				(thickness 0.1)
+			)
+			(justify left bottom)
+		)
+	)
 	(gr_text "165"
 		(at 163.576 84.836 270)
@@
 		)
 	)
+	(gr_text "VGA PMOD Adapter"
+		(at 115.1128 66.548 90)
+		(layer "F.SilkS")
+		(effects
+			(font
+				(size 1.4 1.4)
+				(thickness 0.175)
+			)
+			(justify left bottom)
+		)
+	)
 	(gr_text "b3"
 		(at 162.3568 57.404 0)
@@
 	)
 	(gr_text "< p1"
-		(at 136.34 59.182 0)
+		(at 136.81 59.204 0)
 		(layer "F.SilkS")
 		(effects
@@
 	)
 	(gr_text "R0"
-		(at 131.953 52.324 90)
+		(at 131.826 52.3748 90)
 		(layer "F.SilkS")
 		(effects
@@
 	)
 	(segment
-		(start 159.416 50.676)
-		(end 158.24 49.5)
+		(start 162.052 56.896)
+		(end 159.512 54.356)
 		(width 0.25)
 		(layer "B.Cu")
@@
 	)
 	(segment
-		(start 162.052 56.896)
-		(end 159.416 54.26)
+		(start 159.512 54.356)
+		(end 159.512 50.772)
 		(width 0.25)
 		(layer "B.Cu")
@@
 	)
 	(segment
-		(start 159.416 54.26)
-		(end 159.416 50.676)
+		(start 159.512 50.772)
+		(end 158.24 49.5)
 		(width 0.25)
 		(layer "B.Cu")
@@
 	(segment
 		(start 164.7825 56.9595)
-		(end 162.144 54.321)
+		(end 162.052 54.229)
 		(width 0.25)
 		(layer "B.Cu")
@@
 	)
 	(segment
-		(start 162.144 50.864)
+		(start 162.052 50.772)
 		(end 160.78 49.5)
 		(width 0.25)
@@
 	)
 	(segment
-		(start 162.144 54.321)
-		(end 162.144 50.864)
+		(start 162.052 54.229)
+		(end 162.052 50.772)
 		(width 0.25)
 		(layer "B.Cu")
